File: HPLC/untitled.sch (EAGLE design)
At the start: 17 parts, among them U2 AMS1117, U3 MAX232CSE, X1 MSTBA2, X2 MSTBA4, X4 MSTBA3

Commit message: PCB huawei
Parts:
- added X3: C-GRID-02-70543, con-molex:C-GRID-02-70543
Connections:
- net 5V: now also X3-1.S
- net GND: now also X3-2.S
Changed lines of the file:
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@@
 <part name="X2" library="con-phoenix-508" library_urn="urn:adsk.eagle:library:176" deviceset="MSTBA4" device="" package3d_urn="urn:adsk.eagle:package:9613/1"/>
 <part name="GND2" library="supply1" library_urn="urn:adsk.eagle:library:371" deviceset="GND" device=""/>
+<part name="X3" library="con-molex" library_urn="urn:adsk.eagle:library:165" deviceset="C-GRID-02" device="-70543" package3d_urn="urn:adsk.eagle:package:8078681/1"/>
+<part name="GND8" library="supply1" library_urn="urn:adsk.eagle:library:371" deviceset="GND" device=""/>
 </parts>
 <sheets>
@@
 <attribute name="VALUE" x="203.2" y="55.88" size="1.778" layer="96"/>
 </instance>
+<instance part="X3" gate="-2" x="157.48" y="160.02" smashed="yes" rot="R180">
+<attribute name="NAME" x="154.94" y="160.782" size="1.524" layer="95" rot="R180"/>
+</instance>
+<instance part="X3" gate="-1" x="157.48" y="157.48" smashed="yes" rot="R180">
+<attribute name="NAME" x="154.94" y="158.242" size="1.524" layer="95" rot="R180"/>
+<attribute name="VALUE" x="158.242" y="156.083" size="1.778" layer="96" rot="R180"/>
+</instance>
+<instance part="GND8" gate="1" x="172.72" y="157.48" smashed="yes">
+<attribute name="VALUE" x="170.18" y="154.94" size="1.778" layer="96"/>
+</instance>
 </instances>
 <busses>
@@
 <pinref part="GND2" gate="1" pin="GND"/>
 </segment>
+<segment>
+<pinref part="X3" gate="-2" pin="S"/>
+<pinref part="GND8" gate="1" pin="GND"/>
+<wire x1="160.02" y1="160.02" x2="172.72" y2="160.02" width="0.1524" layer="91"/>
+</segment>
 </net>
 <net name="N$7" class="0">
@@
 <label x="17.78" y="162.56" size="0.6096" layer="95" rot="R90" xref="yes"/>
 </segment>
-</net>
+<segment>
+<pinref part="X3" gate="-1" pin="S"/>
+<wire x1="160.02" y1="157.48" x2="162.56" y2="157.48" width="0.1524" layer="91"/>
+<label x="162.56" y="157.48" size="0.6096" layer="95" xref="yes"/>
+</segment>
+</net>
