File: HPLC/untitled.brd (EAGLE design)
At the start: 100 x 130 mm, 17 parts, among them U2 AMS1117, U3 MAX232CSE, X1 MSTBA2, X2 MSTBA4, X4 MSTBA3

Commit message: PCB huawei
Parts:
- added X3: C-GRID-02-70543, con-molex:70543-02
Connections:
- net 5V: now also X3.1
- net GND: now also X3.2
Routing:
- net 12V: track 184.4 -> 193.6 mm
- net 5V: track 53.3 -> 61.0 mm
Changed lines of the file:
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@@
 <attribute name="VALUE" x="41.137534375" y="1.978915625" size="1.778" layer="27" ratio="10"/>
+</element>
+<element name="X3" library="con-molex" library_urn="urn:adsk.eagle:library:165" package="70543-02" package3d_urn="urn:adsk.eagle:package:8078681/1" value="C-GRID-02-70543" x="92.3729625" y="41.7389375" smashed="yes" rot="R90">
+<attribute name="MF" value="MOLEX" x="92.3729625" y="41.7389375" size="1.778" layer="27" rot="R90" display="off"/>
+<attribute name="MPN" value="" x="92.3729625" y="41.7389375" size="1.778" layer="27" rot="R90" display="off"/>
+<attribute name="NAME" x="94.9129625" y="37.2939375" size="1.016" layer="25" ratio="10" rot="R180"/>
+<attribute name="OC_FARNELL" value="unknown" x="92.3729625" y="41.7389375" size="1.778" layer="27" rot="R90" display="off"/>
+<attribute name="OC_NEWARK" value="unknown" x="92.3729625" y="41.7389375" size="1.778" layer="27" rot="R90" display="off"/>
+<attribute name="POPULARITY" value="1" x="92.3729625" y="41.7389375" size="1.778" layer="27" rot="R90" display="off"/>
+<attribute name="VALUE" x="88.8804625" y="38.2464375" size="0.8128" layer="27" ratio="10" rot="R90"/>
 </element>
 </elements>
@@
 <wire x1="56.261453125" y1="21.178934375" x2="56.22115625" y2="21.1386375" width="0.4064" layer="1"/>
 <via x="56" y="23" extent="1-16" drill="0.35"/>
+<contactref element="X3" pad="2"/>
 </signal>
 <signal name="N$7">
@@
 <wire x1="62.9823625" y1="25.44643125" x2="63.17751875" y2="25.44643125" width="0.508" layer="1"/>
 <wire x1="63.17751875" y1="25.44643125" x2="63.612540625" y2="25.011409375" width="0.508" layer="1"/>
+<contactref element="X3" pad="1"/>
+<wire x1="85.244046875" y1="38.950971875" x2="90.854996875" y2="38.950971875" width="0.508" layer="1"/>
+<wire x1="90.854996875" y1="38.950971875" x2="92.3729625" y2="40.4689375" width="0.508" layer="1"/>
 </signal>
 <signal name="3V3">
@@
 <wire x1="64.307109375" y1="17.6967125" x2="67.514040625" y2="17.6967125" width="0.508" layer="1"/>
 <wire x1="60.9269875" y1="14.316590625" x2="64.307109375" y2="17.6967125" width="0.508" layer="1"/>
-<wire x1="67.514040625" y1="17.6967125" x2="88.8290375" y2="17.6967125" width="0.508" layer="1"/>
-<wire x1="88.8290375" y1="17.6967125" x2="91.4892625" y2="20.3569375" width="0.508" layer="1"/>
-<wire x1="91.4892625" y1="20.3569375" x2="91.4892625" y2="107.416490625" width="0.508" layer="1"/>
-<wire x1="91.4892625" y1="107.416490625" x2="73.044971875" y2="125.86078125" width="0.508" layer="1"/>
-<wire x1="73.044971875" y1="125.86078125" x2="49.29553125" y2="125.86078125" width="0.508" layer="1"/>
+<wire x1="67.514040625" y1="17.6967125" x2="93.047503125" y2="17.6967125" width="0.508" layer="1"/>
+<wire x1="93.047503125" y1="17.6967125" x2="96.714625" y2="21.363834375" width="0.508" layer="1"/>
+<wire x1="96.714625" y1="21.363834375" x2="96.714625" y2="106.431103125" width="0.508" layer="1"/>
+<wire x1="96.714625" y1="106.431103125" x2="77.284946875" y2="125.86078125" width="0.508" layer="1"/>
+<wire x1="77.284946875" y1="125.86078125" x2="49.29553125" y2="125.86078125" width="0.508" layer="1"/>
 <wire x1="46.91915625" y1="123.48440625" x2="46.91915625" y2="122.232315625" width="0.508" layer="1"/>
 <wire x1="49.29553125" y1="125.86078125" x2="46.91915625" y2="123.48440625" width="0.508" layer="1"/>

Commit message: revisi HPLC
Parts:
- moved X3 87.5 mm to (4.90, 42.6), turned to 270 degrees
- moved D5 75.4 mm to (10.0, 39.7), turned to 90 degrees
- moved R5 75.3 mm to (10.0, 44.4), turned to 90 degrees
- moved D2 7.07 mm to (60.5, 14.5)
- moved C10 7.07 mm to (32.9, 23.6)
- moved C11 7.07 mm to (33.0, 19.5)
- moved C12 7.07 mm to (40.1, 27.7)
- moved C8 7.07 mm to (49.2, 19.1)
- moved C9 7.07 mm to (52.2, 19.2)
- moved D3 7.07 mm to (60.5, 28.6)
- moved MINI1 7.07 mm to (64.9, 3.88)
- moved U2 7.07 mm to (51.4, 27.8)
- moved U3 7.07 mm to (39.8, 19.4)
- moved X1 7.00 mm to (56.5, 1.99)
- moved X4 7.00 mm to (41.8, 1.98)
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Routing:
- net 5V: track 61.0 -> 105.3 mm, vias 0 -> 2
- net 12V: track 193.6 -> 159.6 mm
- net PLC-N: track 48.0 -> 52.5 mm
- net PLC-A: track 44.9 -> 42.0 mm
- net TX_RS232: track 109.7 -> 112.3 mm
- net RX_RS232: track 108.4 -> 110.8 mm
- net T2OUT: track 13.9 -> 12.5 mm
- net N$15: track 6.81 -> 5.46 mm
- net PLC-B: track 46.0 -> 44.6 mm
Other:
- board size 100 x 130 mm -> 84 x 125 mm

Commit message: revisi HPLC
Parts:
- moved HUAWEI-PLC1 3.00 mm to (51.7, 122.2)
- moved MINI1 1.00 mm to (64.9, 2.88)
Routing:
- net TX_RS232: track 112.3 -> 107.6 mm
- net RX_RS232: track 110.8 -> 106.2 mm
- net 12V: track 159.6 -> 162.6 mm
- net PLC-C: track 47.0 -> 48.9 mm
- net PLC-A: track 42.0 -> 43.8 mm
- net N$9: track 8.20 -> 7.20 mm
- net N$7: track 13.1 -> 14.1 mm
- net PLC-B: track 44.6 -> 45.6 mm

Commit message: 3 PCB done
Parts:
- moved C13 30.0 mm to (61.5, 11.9), flipped to the bottom
- moved C11 28.9 mm to (61.8, 17.2), flipped to the bottom
- moved C10 28.9 mm to (61.8, 22.0), flipped to the bottom
- moved D2 23.5 mm to (67.8, 36.8), flipped to the bottom
- moved D3 16.5 mm to (74.8, 36.9), flipped to the bottom
- moved MINI1 15.9 mm to (80.8, 2.86), flipped to the bottom
- moved C12 15.4 mm to (55.4, 26.2), flipped to the bottom
- moved U3 15.0 mm to (54.8, 18.8), flipped to the bottom
- moved HUAWEI-PLC1 14.9 mm to (47.9, 107.8)
- moved C8 14.4 mm to (58.7, 30.0), flipped to the bottom
- moved D5 11.6 mm to (4.84, 50.0)
- moved R5 11.6 mm to (4.82, 54.8)
- moved C9 11.3 mm to (55.8, 29.9), flipped to the bottom
- moved U2 11.1 mm to (55.7, 38.1), flipped to the bottom
Routing:
- net 5V: track 105.3 -> 145.4 mm, vias 2 -> 1
- net PLC-N: track 52.2 -> 26.3 mm
- net N$7: track 14.1 -> 39.3 mm
- net PLC-C: track 48.9 -> 25.1 mm
- net PLC-B: track 45.6 -> 24.1 mm
- net PLC-A: track 43.8 -> 23.1 mm
- net TX_RS232: track 107.6 -> 91.4 mm
- net RX_RS232: track 106.2 -> 90.1 mm
- net T2OUT: track 12.5 -> 27.6 mm
- net 3V3: track 40.4 -> 26.4 mm, vias 2 -> 0
- net 12V: track 162.6 -> 150.2 mm, vias 0 -> 1
- net R2IN: track 15.8 -> 21.1 mm
- net N$9: track 7.20 -> 9.27 mm
- net N$15: track 5.46 -> 7.03 mm
- net N$14: track 4.46 -> 5.35 mm
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