File: SUPERCAP/untitled.sch (EAGLE design)
At the start: 69 parts, among them Q1 SS8550, Q10 TSM60NC1R5CP, Q11 SS8550, Q12 TSM60NC1R5CP, Q2 TSM60NC1R5CP, Q3 SS8550, Q4 TSM60NC1R5CP, Q5 SS8550, Q6 TSM60NC1R5CP, Q7 SS8550, Q8 TSM60NC1R5CP, Q9 SS8550, U1 TL431AIDBZT, U4 TL431AIDBZT, U5 TL431AIDBZT, U6 TL431AIDBZT, U7 TL431AIDBZT, U8 TL431AIDBZT, X2 MSTBA4, X3 MSTBA2, X4 MSTBA2

Commit message: PCB SUPERCAP dan HPLC
Parts:
- removed X3: MSTBA2, con-phoenix-508:MSTBA2
- added POWERMETER1: (no value), POWERMETER:POWERMETER
- added X1: MSTBA6, con-phoenix-508:MSTBA6
- added X5: MSTBA2, con-phoenix-508:MSTBA2
- added X6: MSTBA3, con-phoenix-508:MSTBA3
Connections:
- new net A: POWERMETER1.A, X5-1.1
- new net B: POWERMETER1.B, X5-2.1
- new net G: POWERMETER1.G, X6-1.1
- new net IA1: POWERMETER1.I11, X1-6.1
- new net IA2: POWERMETER1.I12, X1-5.1
- new net IB1: POWERMETER1.I21, X1-4.1
- new net IB2: POWERMETER1.I22, X1-3.1
- new net IC1: POWERMETER1.I31, X1-2.1
- new net IC2: POWERMETER1.I32, X1-1.1
- net 12V: now also X4-2.1; no longer X4-1.1
- net GND: now also X4-1.1; no longer X4-2.1
- net NEG(-): now also X6-3.1; no longer X3-2.1
- net PLC-A: now also POWERMETER1.L, POWERMETER1.V1
- net PLC-B: now also POWERMETER1.V2
- net PLC-C: now also POWERMETER1.V3
- net PLC-N: now also POWERMETER1.N, POWERMETER1.VN
- net POS(+): now also X6-2.1; no longer X3-1.1
Other:
- note added: "POWER METER"
- moved on the sheet: X2-1, X2-2, X2-3, X2-4

Commit message: revisi HPLC
Connections:
- net NEG(-): now also POWERMETER1.N
- net PLC-A: no longer POWERMETER1.L
- net PLC-N: no longer POWERMETER1.N
- net POS(+): now also POWERMETER1.L
Changed lines of the file:
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@@
 <label x="83.82" y="99.06" size="0.6096" layer="95" rot="R90" xref="yes"/>
+</segment>
+<segment>
+<pinref part="POWERMETER1" gate="G$1" pin="L"/>
+<wire x1="187.96" y1="137.16" x2="187.96" y2="134.62" width="0.1524" layer="91"/>
+<label x="187.96" y="134.62" size="0.6096" layer="95" rot="R270" xref="yes"/>
 </segment>
 </net>
@@
 <wire x1="88.9" y1="96.52" x2="88.9" y2="99.06" width="0.1524" layer="91"/>
 <label x="88.9" y="99.06" size="0.6096" layer="95" rot="R90" xref="yes"/>
+</segment>
+<segment>
+<pinref part="POWERMETER1" gate="G$1" pin="N"/>
+<wire x1="193.04" y1="137.16" x2="193.04" y2="134.62" width="0.1524" layer="91"/>
+<label x="193.04" y="134.62" size="0.6096" layer="95" rot="R270" xref="yes"/>
 </segment>
 </net>
@@
 <wire x1="15.24" y1="93.98" x2="15.24" y2="96.52" width="0.1524" layer="91"/>
 <label x="15.24" y="96.52" size="0.6096" layer="95" rot="R90" xref="yes"/>
-</segment>
-<segment>
-<pinref part="POWERMETER1" gate="G$1" pin="L"/>
-<wire x1="187.96" y1="137.16" x2="187.96" y2="134.62" width="0.1524" layer="91"/>
-<label x="187.96" y="134.62" size="0.6096" layer="95" rot="R270" xref="yes"/>
 </segment>
 <segment>
@@
 </segment>
 <segment>
-<pinref part="POWERMETER1" gate="G$1" pin="N"/>
-<wire x1="193.04" y1="137.16" x2="193.04" y2="134.62" width="0.1524" layer="91"/>
-<label x="193.04" y="134.62" size="0.6096" layer="95" rot="R270" xref="yes"/>
-</segment>
-<segment>
