File: SUPERCAP/untitled.brd (EAGLE design)
At the start: 100 x 100 mm, 69 parts, among them Q1 SS8550, Q10 TSM60NC1R5CP, Q11 SS8550, Q12 TSM60NC1R5CP, Q2 TSM60NC1R5CP, Q3 SS8550, Q4 TSM60NC1R5CP, Q5 SS8550, Q6 TSM60NC1R5CP, Q7 SS8550, Q8 TSM60NC1R5CP, Q9 SS8550, U1 TL431AIDBZT, U4 TL431AIDBZT, U5 TL431AIDBZT, U6 TL431AIDBZT, U7 TL431AIDBZT, U8 TL431AIDBZT, X2 MSTBA4, X3 MSTBA2, X4 MSTBA2

Commit message: revisi HPLC
Parts:
- moved R29 410.3 mm to (75.2, 68.0), flipped to the bottom, turned to 270 degrees
- moved R30 409.2 mm to (81.4, 68.0), flipped to the bottom, turned to 270 degrees
- moved R31 408.4 mm to (88.3, 67.9), flipped to the bottom, turned to 270 degrees
- moved R26 390.3 mm to (92.8, 51.7), flipped to the bottom, turned to 90 degrees
- moved R27 389.6 mm to (84.4, 51.8), flipped to the bottom, turned to 90 degrees
- moved R28 386.9 mm to (88.9, 51.8), flipped to the bottom, turned to 90 degrees
- moved SUPERCAP6 385.5 mm to (78.5, 21.3), turned to 180 degrees
- moved Q10 383.6 mm to (75.2, 50.1), flipped to the bottom
- moved U7 377.4 mm to (84.1, 45.5), flipped to the bottom
- moved Q9 369.4 mm to (90.1, 45.6), flipped to the bottom, turned to 270 degrees
- moved SUPERCAP5 367.4 mm to (85.7, 54.2)
- moved SUPERCAP4 284.3 mm to (14.7, 48.8), turned to 180 degrees
- moved SUPERCAP3 239.9 mm to (49.3, 41.1), turned to 180 degrees
- moved SUPERCAP2 209.5 mm to (22.2, 77.1)
- moved SUPERCAP1 201.1 mm to (59.0, 78.5)
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Routing:
- net NEG(-): track 0.00 -> 63.8 mm
- net POS(+): track 0.00 -> 54.4 mm
- net PLC-N: track 0.00 -> 54.1 mm
- net N$45: track 0.00 -> 43.9 mm
- net CAP1-: track 0.00 -> 43.6 mm
- net CAP2-: track 0.00 -> 28.8 mm, vias 0 -> 1
- net N$41: track 0.00 -> 25.1 mm, vias 0 -> 3
- net PLC-A: track 0.00 -> 22.9 mm
- net N$44: track 0.00 -> 15.5 mm, vias 0 -> 2
- net PLC-B: track 0.00 -> 15.1 mm
- net PLC-C: track 0.00 -> 14.0 mm
- net N$43: track 0.00 -> 11.2 mm
- net N$1: track 0.00 -> 6.37 mm
- net N$2: track 0.00 -> 5.99 mm
- net N$3: track 0.00 -> 5.75 mm

Commit message: PCB SUPERCAP dan HPLC
Parts:
- removed X3: MSTBA2, con-phoenix-508:MSTBA2
- added POWERMETER1: (no value), POWERMETER:POWERMETER
- added X1: MSTBA6, con-phoenix-508:MSTBA6
- added X5: MSTBA2, con-phoenix-508:MSTBA2
- added X6: MSTBA3, con-phoenix-508:MSTBA3
- moved R35 428.0 mm to (82.6, 28.3), flipped to the bottom, turned to 270 degrees
- moved R36 427.6 mm to (90.3, 28.3), flipped to the bottom, turned to 270 degrees
- moved R37 418.9 mm to (75.9, 28.3), flipped to the bottom, turned to 270 degrees
- moved R32 403.4 mm to (92.3, 10.2), flipped to the bottom, turned to 90 degrees
- moved R33 402.8 mm to (84.0, 10.3), flipped to the bottom, turned to 90 degrees
- moved R34 400.0 mm to (87.6, 10.4), flipped to the bottom, turned to 90 degrees
- moved Q12 395.5 mm to (73.7, 7.89), flipped to the bottom
- moved U8 391.6 mm to (84.5, 4.99), flipped to the bottom
- moved Q11 383.7 mm to (90.5, 4.95), flipped to the bottom, turned to 270 degrees
- moved R23 327.7 mm to (25.4, 54.9), flipped to the bottom, turned to 270 degrees
- moved R24 322.7 mm to (18.7, 54.9), flipped to the bottom, turned to 270 degrees
- moved R25 318.4 mm to (12.3, 54.8), flipped to the bottom, turned to 270 degrees
- moved R20 302.7 mm to (27.1, 38.0), flipped to the bottom, turned to 90 degrees
- moved R21 301.7 mm to (17.3, 38.0), flipped to the bottom, turned to 90 degrees
- moved R22 299.9 mm to (21.9, 37.9), flipped to the bottom, turned to 90 degrees
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Connections:
- new net A: POWERMETER1.A, X5.1
- new net B: POWERMETER1.B, X5.2
- new net G: POWERMETER1.G, X6.1
- new net IA1: POWERMETER1.I11, X1.6
- new net IA2: POWERMETER1.I12, X1.5
- new net IB1: POWERMETER1.I21, X1.4
- new net IB2: POWERMETER1.I22, X1.3
- new net IC1: POWERMETER1.I31, X1.2
- new net IC2: POWERMETER1.I32, X1.1
- net 12V: now also X4.2; no longer X4.1
- net GND: now also X4.1; no longer X4.2
- net NEG(-): now also X6.3; no longer X3.2
- net PLC-A: now also POWERMETER1.L, POWERMETER1.V1
- net PLC-B: now also POWERMETER1.V2
- net PLC-C: now also POWERMETER1.V3
- net PLC-N: now also POWERMETER1.N, POWERMETER1.VN
- net POS(+): now also X6.2; no longer X3.1
Routing:
- net PLC-A: track 22.9 -> 230.4 mm, vias 0 -> 1
- net PLC-C: track 14.0 -> 216.5 mm
- net PLC-N: track 54.1 -> 238.6 mm, vias 0 -> 1
- net PLC-B: track 15.1 -> 166.4 mm
- net GND: track 0.00 -> 145.6 mm, vias 0 -> 1
- net CAP4-: track 0.00 -> 136.1 mm, vias 0 -> 2
- net CAP5-: track 0.00 -> 127.4 mm, vias 0 -> 2
- net G: track 0.00 -> 120.4 mm
- net CAP3-: track 0.00 -> 104.7 mm, vias 0 -> 1
- net A: track 0.00 -> 100.5 mm
- net B: track 0.00 -> 95.2 mm
- net 12V: track 0.00 -> 82.0 mm
- net CAP1-: track 43.6 -> 125.1 mm
- net CAP2-: track 28.8 -> 95.9 mm, vias 1 -> 2
- net N$51: track 0.00 -> 47.9 mm
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- added copper zone on layer 1, net GND
- added copper zone on layer 16, net GND
Other:
- board size 100 x 100 mm -> 186 x 98 mm

Commit message: revisi HPLC
Connections:
- net NEG(-): now also POWERMETER1.N
- net PLC-A: no longer POWERMETER1.L
- net PLC-N: no longer POWERMETER1.N
- net POS(+): now also POWERMETER1.L
Routing:
- net NEG(-): track 62.6 -> 170.1 mm
- net POS(+): track 79.4 -> 178.0 mm
- net PLC-A: track 230.4 -> 148.5 mm
- net PLC-N: track 238.6 -> 197.2 mm
- net G: track 120.4 -> 118.3 mm
