File: LED/untitled.brd (EAGLE design)
At the start: 84.3 x 19.3 mm, 7 parts, among them X1 C-GRID-04-70543

Commit message: REVISI PCB LED
Parts:
- moved LED1 3.74 mm to (62.0, 9.50)
- moved LED2 2.25 mm to (42.0, 9.50)
- moved R1 1.71 mm to (66.6, 9.04)
- moved R2 1.18 mm to (47.6, 8.91)
- moved LED3 0.90 mm to (22.1, 9.50)
Connections:
- net GND: no longer LED1.C, LED2.C
- net N$1: now also LED2.C, X1.3; no longer R1.1, X1.4
- net N$2: now also LED1.C, X1.4; no longer R2.1, X1.3
- net N$3: now also R1.1, R2.1
Routing:
- net GND: track 88.3 -> 19.0 mm
- net N$3: track 15.4 -> 79.8 mm
- net N$1: track 26.2 -> 5.43 mm
- net N$2: track 9.63 -> 21.9 mm
- net N$4: track 6.79 -> 4.66 mm
- net N$5: track 6.95 -> 5.68 mm
- net N$6: track 6.72 -> 5.76 mm
